File: ROV_Schematics_NoPCB.kicad_sch (KiCad schematic)
At the start: 7 parts

Commit message: Jetson Nano power
Other:
- note added: "Only includes needed pins of dev kit"
- note removed: "Only includes needed pins of dev kit (below)"
